Commit message: 0706_localization_mode

File: install_isolated/share/cartographer_ros/urdf/my_robot.urdf (robot description, URDF)
Before this commit: robot myrobot, 2 links, 1 joints
Links:
- removed link base_laser
- added link laser_link; visual cylinder length=0.05 radius=0.03
Joints:
- removed joint base_laser
- added joint base_laser_joint: type fixed, parent base_link, child laser_link, origin xyz=0 0 0

Commit message: 0710 지도 다시 작성, tf 구조 수정

File: install_isolated/share/cartographer_ros/urdf/my_robot.urdf (robot description, URDF)
Before this commit: robot myrobot, 2 links, 1 joints
Links:
- removed link laser_link
- added link laser; visual cylinder length=0.05 radius=0.03
- added link odom; visual cylinder length=0.05 radius=0.03
Joints:
- added joint odom_base_joint: type fixed, parent odom, child base_link, origin xyz=0 0 0
- joint base_laser_joint: child laser_link -> laser
